File: pmon_uno/eagle/cover_top.brd (EAGLE design)
At the start: 60 x 60 mm, 0 parts

Commit message: Changed the button and power terminals to be top access (incremented to Rev B), Yet to be auto routed.
Changed lines of the file:
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@@
 <setting verticaltext="up"/>
 </settings>
-<grid distance="5" unitdist="mm" unit="mm" style="lines" multiple="1" display="yes" altdistance="0.025" altunitdist="inch" altunit="inch"/>
+<grid distance="100" unitdist="mil" unit="mil" style="lines" multiple="1" display="yes" altdistance="0.025" altunitdist="inch" altunit="inch"/>
 <layers>
 <layer number="1" name="Top" color="4" fill="1" visible="no" active="yes"/>
@@
 <board>
 <plain>
-<wire x1="0" y1="-5" x2="50" y2="-5" width="0" layer="20"/>
-<wire x1="55" y1="0" x2="55" y2="50" width="0" layer="20"/>
-<wire x1="50" y1="55" x2="0" y2="55" width="0" layer="20"/>
-<wire x1="-5" y1="50" x2="-5" y2="0" width="0" layer="20"/>
-<wire x1="-5" y1="0" x2="0" y2="-5" width="0" layer="20" curve="90"/>
+<wire x1="0" y1="-5" x2="50" y2="-5" width="0.0254" layer="20"/>
+<wire x1="55" y1="0" x2="55" y2="50" width="0.0254" layer="20"/>
+<wire x1="50" y1="55" x2="0" y2="55" width="0.0254" layer="20"/>
+<wire x1="-5" y1="50" x2="-5" y2="0" width="0.0254" layer="20"/>
+<wire x1="-5" y1="0" x2="0" y2="-5" width="0.0254" layer="20" curve="90"/>
 <wire x1="0" y1="55" x2="-5" y2="50" width="0" layer="20" curve="90"/>
-<wire x1="55" y1="50" x2="50" y2="55" width="0" layer="20" curve="90"/>
-<wire x1="50" y1="-5" x2="55" y2="0" width="0" layer="20" curve="90"/>
+<wire x1="55" y1="50" x2="50" y2="55" width="0.0254" layer="20" curve="90"/>
+<wire x1="50" y1="-5" x2="55" y2="0" width="0.0254" layer="20" curve="90"/>
 <hole x="4" y="4" drill="2.5"/>
 <hole x="46" y="4" drill="2.5"/>
