File: pmon_uno/eagle/pmon_uno.brd (EAGLE design)
At the start: 50 x 50 mm, 43 parts, among them J1 USB, J2 USB, J3 PINHD-1X3, J4 PINHD-2X3, J5 PINHD-1X3, Q1 16Mhz, U1 LTC2943, U2 FT232RL, U3 LT1764AEQ, U4 ATMEGA328TQFP32

Commit message: Changed reset capacitor from 0.01 to 0.1 (to reduce compoent kind count).
Parts:
- C7: value 0.01uF -> 0.1uF
Changed lines of the file:
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@@
 <attribute name="NAME" x="13.081" y="9.271" size="0.762" layer="25" font="vector" ratio="10"/>
 </element>
-<element name="C7" library="pmon_uno" package="C0603" value="0.01uF" x="11.049" y="27.305" smashed="yes" rot="R270">
+<element name="C7" library="pmon_uno" package="C0603" value="0.1uF" x="11.049" y="27.305" smashed="yes" rot="R270">
 <attribute name="NAME" x="12.954" y="26.8605" size="0.762" layer="25" font="vector" ratio="10" rot="R90"/>
 </element>
