File: pmon_5v/eagle/pmon_5v.brd (EAGLE design)
At the start: 60 x 60 mm, 30 parts, among them J1 USB, J2 USB, J4 USB_A, J5 PINHD-2X3, Q1 16Mhz, U1 LTC2943, U2 FT232RL, U4 ATMEGA328TQFP32

Commit message: Performed the final auto routing.
Routing:
- net START: track 0.00 -> 40.0 mm, vias 0 -> 2
- net RESET: track 0.00 -> 37.9 mm
- net MISO: track 0.12 -> 34.8 mm, vias 0 -> 2
- net SCK: track 0.30 -> 34.9 mm
- net MOSI: track 0.11 -> 34.7 mm, vias 0 -> 1
- net I2C-DATA: track 0.00 -> 24.7 mm, vias 0 -> 3
- net SER_RX: track 0.00 -> 23.9 mm, vias 0 -> 2
- net I2C-CLK: track 0.13 -> 17.9 mm, vias 0 -> 2
- net N$8: track 0.00 -> 16.1 mm
- net N$1: track 0.05 -> 12.0 mm, vias 0 -> 2
- net N$6: track 0.00 -> 8.10 mm
- net SER_TX: track 0.00 -> 8.03 mm
- net GND: track 72.2 -> 74.4 mm
- net N$4: track 0.00 -> 2.00 mm

Commit message: Cleaned up the board.
Parts:
- removed C12: 20pF, pmon_5v:C0603
- removed J5: PINHD-2X3, pmon_5v:2X03
- added C8: 0.1uF, pmon_5v:C0603
- added J3: USB_A, pmon_5v:USB_A
- C10: value 0.1uF -> 20pF
- C3: value 10uF -> 0.1uF; device pmon_5v:A/3216-18R -> pmon_5v:C0603
- C4: value 0.1uF -> 10uF; device pmon_5v:C0603 -> pmon_5v:A/3216-18R
- J4: value USB_A -> PINHD-2X3; device pmon_5v:USB_A -> pmon_5v:2X03
- R4: value 10K -> 0.025R 1%; device pmon_5v:R0603 -> pmon_5v:KELVIN-6432
- R6: value 0.025R 1% -> 10K; device pmon_5v:KELVIN-6432 -> pmon_5v:R0603
- moved R4 47.1 mm to (51.6, 39.4), turned to 90 degrees
- moved J4 44.7 mm to (4.12, 26.7)
- moved R6 35.4 mm to (17.1, 47.6), turned to 270 degrees
- moved C5 34.6 mm to (46.4, 48.4)
- moved C3 31.6 mm to (12.1, 53.3), turned to 90 degrees
- moved J1 24.0 mm to (18.0, 60.5)
- moved J2 24.0 mm to (42.0, 60.5)
- moved R5 18.8 mm to (4.80, 33.4), turned to 180 degrees
- moved C10 15.6 mm to (17.1, 35.6), turned to 0 degrees
- moved C4 3.05 mm to (43.3, 48.5), turned to 270 degrees
- renumbered C11 to C9, R10 to R7, R11 to R8, U4 to U3
Connections:
- net +5V: now also C4.+, C5.1, C8.1, J2.1, J4.2, R4.I2; no longer C10.1, C3.+, C4.1, J1.1, J5.2, R6.I2
- net GND: now also C3.2, C4.-, C8.2, J3.4, J4.6; no longer C12.2, C3.-, C4.2, J4.4, J5.6
- net MISO: now also J4.1; no longer J5.1
- net MOSI: now also J4.4; no longer J5.4
- net N$10: now also J1.3; no longer J2.3
- net N$15: now also J1.2; no longer J2.2
- net N$22: now also J3.1, R4.I1; no longer J4.1, R6.I1
- net N$4: now also J3.2, J3.3; no longer J4.2, J4.3
- net N$6: now also R5.2; no longer R4.2
- net N$7: now also C10.1; no longer C12.1
- net N$8: now also R6.2; no longer R5.2
- net RESET: now also J4.5; no longer J5.5
- net SCK: now also J4.3; no longer J5.3
- net SENSE+: now also R4.V2; no longer R6.V2
- net SENSE-: now also R4.V1; no longer R6.V1
- net SER_RX: now also R5.1; no longer R4.1
- net SER_TX: now also R6.1; no longer R5.1
- net VUSB: now also C3.1, J1.1; no longer C5.1, J2.1
Routing:
- net N$4: track 2.00 -> 7.57 mm
