File: pmon_5v/eagle/cover_top.brd (EAGLE design)
At the start: 66 x 66 mm, 4 parts, among them J1 USB, J2 USB

Commit message: Updated laser cut design files.
Parts:
- removed JP1: (no value), pmon_oled:1X03
- added U$2: USB_A, pmon_5v:USB_A
- J1, J2: device pmon_3v8:USB-MICRO-ZX62RD-AB-5P8 -> pmon_5v:USB-MICRO-ZX62RD-AB-5P8
Other:
- outline, holes or cut-outs redrawn
- board text added: "POWER-PLAY 5V"
- board text removed: "POWER-PLAY 3.8V"
Changed lines of the file:
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@@
 <setting verticaltext="up"/>
 </settings>
-<grid distance="196.850394" unitdist="mil" unit="mil" style="lines" multiple="1" display="yes" altdistance="1" altunitdist="mil" altunit="mil"/>
+<grid distance="5" unitdist="mil" unit="mil" style="lines" multiple="1" display="yes" altdistance="1" altunitdist="mil" altunit="mil"/>
 <layers>
 <layer number="1" name="Top" color="4" fill="1" visible="yes" active="yes"/>
@@
 <wire x1="56" y1="0" x2="60" y2="4" width="0" layer="48" style="shortdash" curve="90"/>
 <hole x="4.2977375" y="16.99769375" drill="4"/>
-<wire x1="44.961809375" y1="1.56336875" x2="44.961809375" y2="9.38656875" width="0.0254" layer="20"/>
-<wire x1="44.961809375" y1="9.38656875" x2="47.908209375" y2="9.38656875" width="0.0254" layer="20"/>
-<wire x1="47.908209375" y1="9.38656875" x2="47.908209375" y2="1.56336875" width="0.0254" layer="20"/>
-<wire x1="47.908209375" y1="1.56336875" x2="44.961809375" y2="1.56336875" width="0.0254" layer="20"/>
-<text x="42" y="55" size="2.5" layer="20" font="vector" ratio="5" align="bottom-center">USB</text>
-<text x="18" y="55" size="2.5" layer="20" font="vector" ratio="5" align="bottom-center">+5V</text>
-<text x="3" y="40" size="3.1" layer="20" font="vector" ratio="5">POWER-PLAY 3.8V</text>
-<text x="44" y="1.7018" size="2.5" layer="20" font="vector" ratio="5" align="bottom-right">DEVICE</text>
-<text x="70.96" y="28.598" size="1.778" layer="16">NOTE: export the 'dimension' layer only
+<text x="42" y="55" size="2.5" layer="20" font="vector" ratio="10" align="bottom-center">USB</text>
+<text x="18" y="55" size="2.5" layer="20" font="vector" ratio="10" align="bottom-center">+5V</text>
+<text x="3" y="40" size="3.1" layer="20" font="vector" ratio="5">POWER-PLAY 5V</text>
+<text x="59.944" y="19.9898" size="2.5" layer="20" font="vector" ratio="10" rot="SR0" align="bottom-right">DEVICE</text>
+<text x="67.691" y="25.908" size="1.778" layer="16">NOTE: export the 'dimension' layer only
 for laser cut and engraving.</text>
 </plain>
@@
 </autorouter>
 <elements>
-<element name="JP1" library="pmon_oled" package="1X03" value="" x="46.435" y="5.475" rot="R90"/>
 <element name="U$1" library="pmon_oled" package="TLE1105" value="PUSH_BUTTON" x="4.2977375" y="16.99769375" smashed="yes">
 <attribute name="VALUE" x="9.3777375" y="14.45769375" size="1.27" layer="27" rot="R90"/>
 </element>
-<element name="J1" library="pmon_3v8" package="USB-MICRO-ZX62RD-AB-5P8" value="USB" x="17.9832" y="60.5028" smashed="yes" rot="R180"/>
-<element name="J2" library="pmon_3v8" package="USB-MICRO-ZX62RD-AB-5P8" value="USB" x="41.9862" y="60.5028" smashed="yes" rot="R180"/>
+<element name="U$2" library="pmon_5v" package="USB_A" value="USB_A" x="48.4886" y="21.209" rot="R90"/>
+<element name="J1" library="pmon_5v" package="USB-MICRO-ZX62RD-AB-5P8" value="USB" x="17.9832" y="60.5028" smashed="yes" rot="R180"/>
+<element name="J2" library="pmon_5v" package="USB-MICRO-ZX62RD-AB-5P8" value="USB" x="41.9862" y="60.5028" smashed="yes" rot="R180"/>
 </elements>
 <signals>
