File: breakouts/atmega328_breakout/atmega328_breakout.brd (EAGLE design)
At the start: 25.4 x 25.4 mm, 33 parts, among them Q1 16Mhz, U1 ATMEGA328TQFP32

Commit message: Performed final routing.
Routing:
- net RESET: track 0.00 -> 45.5 mm, vias 0 -> 6
- net PD1: track 0.00 -> 27.7 mm, vias 0 -> 4
- net PD6: track 0.00 -> 27.3 mm, vias 0 -> 4
- net PB5: track 0.00 -> 25.6 mm, vias 0 -> 3
- net PC6: track 0.00 -> 25.1 mm, vias 0 -> 2
- net PD7: track 0.00 -> 25.0 mm, vias 0 -> 4
- net PD0: track 0.00 -> 24.1 mm, vias 0 -> 1
- net PD2: track 0.00 -> 24.0 mm, vias 0 -> 3
- net PB4: track 0.00 -> 24.0 mm, vias 0 -> 2
- net PB3: track 0.00 -> 23.9 mm, vias 0 -> 4
- net PC7: track 0.00 -> 22.7 mm, vias 0 -> 2
- net PD5: track 0.00 -> 22.2 mm, vias 0 -> 5
- net PD4: track 0.00 -> 20.3 mm, vias 0 -> 3
- net PB0: track 0.00 -> 18.8 mm, vias 0 -> 4
- net PC5: track 0.00 -> 18.6 mm, vias 0 -> 1
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Other:
- outline, holes or cut-outs redrawn
