File: prototyping/micro_sd_breakout/micro_sd_breakout.brd (EAGLE design)
At the start: 19.1 x 25.4 mm, 9 parts, among them U1 microSD

Commit message: Final routing of the microSD breakout board.
Parts:
- JP1, JP2, JP3, JP4, JP5, JP6, JP7, JP8: device atmega328_breakout:1X01 -> micro_sd_breakout:1X01
- U1: device SparkFun:MICRO-SD-SOCKET-PP -> micro_sd_breakout:MICRO-SD-SOCKET-PP
- moved JP4 2.54 mm to (15.2, 25.4)
- moved JP6 2.54 mm to (12.7, 2.54)
- moved JP7 2.54 mm to (15.2, 2.54)
- moved JP2 2.54 mm to (7.62, 25.4)
- moved JP5 2.54 mm to (10.2, 25.4)
- moved U1 0.64 mm to (16.4, 21.0)
Routing:
- net GND: track 0.00 -> 22.9 mm
- net CD2: track 0.00 -> 17.6 mm
- net SCK: track 0.00 -> 17.1 mm, vias 0 -> 2
- net CS: track 0.00 -> 16.5 mm, vias 0 -> 2
- net VCC: track 0.00 -> 15.5 mm
- net MOSI: track 0.00 -> 13.8 mm, vias 0 -> 2
- net CD1: track 0.00 -> 12.0 mm
- net MISO: track 0.00 -> 9.45 mm
Other:
- board size 19.1 x 25.4 mm -> 17.8 x 25.4 mm
- board text added: "Github OSH"
- board text added: "PRT-00127"
- board text added: "REV1"
- board text added: "WM19114CT-ND"
- board text added: "microSD"
