File: prototyping/micro_sd_breakout/micro_sd_breakout.sch (EAGLE design)
At the start: 9 parts, among them U1 microSD

Commit message: Final routing of the microSD breakout board.
Parts:
- JP1, JP2, JP3, JP4, JP5, JP6, JP7, JP8: device atmega328_breakout:PINHD-1X1 -> micro_sd_breakout:PINHD-1X1
- U1: device SparkFun:USD-SOCKETSMD -> micro_sd_breakout:USD-SOCKETSMD
Other:
- moved on the sheet: U1
Changed lines of the file:
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@@
 <layer number="2" name="Route2" color="1" fill="3" visible="no" active="no"/>
 <layer number="3" name="Route3" color="4" fill="3" visible="no" active="no"/>
-<layer number="4" name="Route4" color="1" fill="4" visible="no" active="no"/>
-<layer number="5" name="Route5" color="4" fill="4" visible="no" active="no"/>
-<layer number="6" name="Route6" color="1" fill="8" visible="no" active="no"/>
-<layer number="7" name="Route7" color="4" fill="8" visible="no" active="no"/>
-<layer number="8" name="Route8" color="1" fill="2" visible="no" active="no"/>
-<layer number="9" name="Route9" color="4" fill="2" visible="no" active="no"/>
-<layer number="10" name="Route10" color="1" fill="7" visible="no" active="no"/>
-<layer number="11" name="Route11" color="4" fill="7" visible="no" active="no"/>
-<layer number="12" name="Route12" color="1" fill="5" visible="no" active="no"/>
-<layer number="13" name="Route13" color="4" fill="5" visible="no" active="no"/>
 <layer number="14" name="Route14" color="1" fill="6" visible="no" active="no"/>
 <layer number="15" name="Route15" color="4" fill="6" visible="no" active="no"/>
@@
 </classes>
 <parts>
-<part name="U1" library="SparkFun" deviceset="USD-SOCKET" device="SMD" value="microSD"/>
-<part name="JP1" library="atmega328_breakout" deviceset="PINHD-1X1" device=""/>
-<part name="U$20" library="atmega328_breakout" deviceset="DOCFIELD" device=""/>
-<part name="JP2" library="atmega328_breakout" deviceset="PINHD-1X1" device=""/>
-<part name="JP3" library="atmega328_breakout" deviceset="PINHD-1X1" device=""/>
-<part name="JP4" library="atmega328_breakout" deviceset="PINHD-1X1" device=""/>
-<part name="JP6" library="atmega328_breakout" deviceset="PINHD-1X1" device=""/>
-<part name="JP7" library="atmega328_breakout" deviceset="PINHD-1X1" device=""/>
-<part name="JP8" library="atmega328_breakout" deviceset="PINHD-1X1" device=""/>
-<part name="JP5" library="atmega328_breakout" deviceset="PINHD-1X1" device=""/>
+<part name="U1" library="micro_sd_breakout" deviceset="USD-SOCKET" device="SMD" value="microSD"/>
+<part name="JP1" library="micro_sd_breakout" deviceset="PINHD-1X1" device=""/>
+<part name="U$20" library="micro_sd_breakout" deviceset="DOCFIELD" device=""/>
+<part name="JP2" library="micro_sd_breakout" deviceset="PINHD-1X1" device=""/>
+<part name="JP3" library="micro_sd_breakout" deviceset="PINHD-1X1" device=""/>
+<part name="JP4" library="micro_sd_breakout" deviceset="PINHD-1X1" device=""/>
+<part name="JP6" library="micro_sd_breakout" deviceset="PINHD-1X1" device=""/>
+<part name="JP7" library="micro_sd_breakout" deviceset="PINHD-1X1" device=""/>
+<part name="JP8" library="micro_sd_breakout" deviceset="PINHD-1X1" device=""/>
+<part name="JP5" library="micro_sd_breakout" deviceset="PINHD-1X1" device=""/>
 </parts>
 <sheets>
@@
 <plain>
 <text x="88.9" y="30.48" size="2.54" layer="97" font="vector">MICRO SD BREAKOUT BOARD</text>
-<wire x1="185.42" y1="154.94" x2="185.42" y2="2.54" width="0.1524" layer="94"/>
-<wire x1="185.42" y1="2.54" x2="0" y2="0" width="0.1524" layer="94"/>
-<text x="177.038" y="9.652" size="2.54" layer="97">1</text>
-<wire x1="185.42" y1="154.94" x2="0" y2="154.94" width="0.1524" layer="94"/>
-<wire x1="0" y1="154.94" x2="0" y2="0" width="0.1524" layer="94"/>
+<wire x1="185.42" y1="124.46" x2="185.42" y2="0" width="0.1524" layer="94"/>
+<wire x1="185.42" y1="0" x2="0" y2="0" width="0.1524" layer="94"/>
+<text x="177.038" y="7.112" size="2.54" layer="97">1</text>
+<wire x1="185.42" y1="124.46" x2="0" y2="124.46" width="0.1524" layer="94"/>
+<wire x1="0" y1="124.46" x2="0" y2="0" width="0.1524" layer="94"/>
 </plain>
 <instances>
-<instance part="U1" gate="G$1" x="55.88" y="93.98" smashed="yes" rot="MR0">
-<attribute name="NAME" x="50.546" y="109.982" size="1.778" layer="95"/>
-<attribute name="VALUE" x="46.736" y="70.866" size="1.778" layer="96"/>
+<instance part="U1" gate="G$1" x="53.34" y="76.2" smashed="yes" rot="MR0">
+<attribute name="NAME" x="48.006" y="92.202" size="1.778" layer="95"/>
+<attribute name="VALUE" x="44.196" y="53.086" size="1.778" layer="96"/>
 </instance>
-<instance part="JP1" gate="G$1" x="88.9" y="104.14" smashed="yes"/>
-<instance part="U$20" gate="G$1" x="83.82" y="2.54"/>
-<instance part="JP2" gate="G$1" x="88.9" y="101.6" smashed="yes"/>
-<instance part="JP3" gate="G$1" x="88.9" y="99.06" smashed="yes"/>
-<instance part="JP4" gate="G$1" x="88.9" y="96.52" smashed="yes"/>
-<instance part="JP6" gate="G$1" x="88.9" y="83.82" smashed="yes"/>
-<instance part="JP7" gate="G$1" x="88.9" y="81.28" smashed="yes"/>
-<instance part="JP8" gate="G$1" x="88.9" y="76.2" smashed="yes"/>
-<instance part="JP5" gate="G$1" x="88.9" y="91.44" smashed="yes"/>
+<instance part="JP1" gate="G$1" x="86.36" y="86.36" smashed="yes"/>
+<instance part="U$20" gate="G$1" x="83.82" y="0"/>
+<instance part="JP2" gate="G$1" x="86.36" y="83.82" smashed="yes"/>
+<instance part="JP3" gate="G$1" x="86.36" y="81.28" smashed="yes"/>
+<instance part="JP4" gate="G$1" x="86.36" y="78.74" smashed="yes"/>
+<instance part="JP6" gate="G$1" x="86.36" y="66.04" smashed="yes"/>
+<instance part="JP7" gate="G$1" x="86.36" y="63.5" smashed="yes"/>
+<instance part="JP8" gate="G$1" x="86.36" y="58.42" smashed="yes"/>
+<instance part="JP5" gate="G$1" x="86.36" y="73.66" smashed="yes"/>
 </instances>
 <busses>
@@
 <net name="CS" class="0">
 <segment>
-<wire x1="63.5" y1="104.14" x2="86.36" y2="104.14" width="0.1524" layer="91"/>
+<wire x1="60.96" y1="86.36" x2="83.82" y2="86.36" width="0.1524" layer="91"/>
 <pinref part="U1" gate="G$1" pin="CS"/>
 <pinref part="JP1" gate="G$1" pin="1"/>
-<label x="73.66" y="104.14" size="1.778" layer="95"/>
+<label x="71.12" y="86.36" size="1.778" layer="95"/>
 </segment>
 </net>
 <net name="MOSI" class="0">
 <segment>
-<wire x1="63.5" y1="101.6" x2="86.36" y2="101.6" width="0.1524" layer="91"/>
+<wire x1="60.96" y1="83.82" x2="83.82" y2="83.82" width="0.1524" layer="91"/>
 <pinref part="U1" gate="G$1" pin="DI"/>
 <pinref part="JP2" gate="G$1" pin="1"/>
-<label x="73.66" y="101.6" size="1.778" layer="95"/>
+<label x="71.12" y="83.82" size="1.778" layer="95"/>
 </segment>
 </net>
 <net name="VCC" class="0">
 <segment>
-<wire x1="63.5" y1="99.06" x2="86.36" y2="99.06" width="0.1524" layer="91"/>
+<wire x1="60.96" y1="81.28" x2="83.82" y2="81.28" width="0.1524" layer="91"/>
 <pinref part="U1" gate="G$1" pin="VCC"/>
 <pinref part="JP3" gate="G$1" pin="1"/>
-<label x="73.66" y="99.06" size="1.778" layer="95"/>
+<label x="71.12" y="81.28" size="1.778" layer="95"/>
 </segment>
 </net>
 <net name="SCK" class="0">
 <segment>
-<wire x1="63.5" y1="96.52" x2="86.36" y2="96.52" width="0.1524" layer="91"/>
+<wire x1="60.96" y1="78.74" x2="83.82" y2="78.74" width="0.1524" layer="91"/>
 <pinref part="U1" gate="G$1" pin="SCK"/>
 <pinref part="JP4" gate="G$1" pin="1"/>
-<label x="73.66" y="96.52" size="1.778" layer="95"/>
+<label x="71.12" y="78.74" size="1.778" layer="95"/>
 </segment>
 </net>
 <net name="GND" class="0">
 <segment>
-<wire x1="63.5" y1="93.98" x2="68.58" y2="93.98" width="0.1524" layer="91"/>
-<wire x1="63.5" y1="76.2" x2="68.58" y2="76.2" width="0.1524" layer="91"/>
-<wire x1="68.58" y1="76.2" x2="68.58" y2="78.74" width="0.1524" layer="91"/>
-<wire x1="68.58" y1="78.74" x2="68.58" y2="93.98" width="0.1524" layer="91"/>
-<wire x1="63.5" y1="78.74" x2="68.58" y2="78.74" width="0.1524" layer="91"/>
-<junction x="68.58" y="78.74"/>
+<wire x1="60.96" y1="76.2" x2="66.04" y2="76.2" width="0.1524" layer="91"/>
+<wire x1="60.96" y1="58.42" x2="66.04" y2="58.42" width="0.1524" layer="91"/>
+<wire x1="66.04" y1="58.42" x2="66.04" y2="60.96" width="0.1524" layer="91"/>
+<wire x1="66.04" y1="60.96" x2="66.04" y2="76.2" width="0.1524" layer="91"/>
+<wire x1="60.96" y1="60.96" x2="66.04" y2="60.96" width="0.1524" layer="91"/>
+<junction x="66.04" y="60.96"/>
 <pinref part="U1" gate="G$1" pin="GND"/>
 <pinref part="U1" gate="G$1" pin="SHIELD1"/>
 <pinref part="U1" gate="G$1" pin="SHIELD2"/>
 <pinref part="JP8" gate="G$1" pin="1"/>
-<wire x1="68.58" y1="76.2" x2="86.36" y2="76.2" width="0.1524" layer="91"/>
-<label x="73.66" y="76.2" size="1.778" layer="95"/>
-<junction x="68.58" y="76.2"/>
+<wire x1="66.04" y1="58.42" x2="83.82" y2="58.42" width="0.1524" layer="91"/>
+<label x="71.12" y="58.42" size="1.778" layer="95"/>
+<junction x="66.04" y="58.42"/>
 </segment>
 </net>
 <net name="MISO" class="0">
 <segment>
-<wire x1="63.5" y1="91.44" x2="86.36" y2="91.44" width="0.1524" layer="91"/>
+<wire x1="60.96" y1="73.66" x2="83.82" y2="73.66" width="0.1524" layer="91"/>
 <pinref part="U1" gate="G$1" pin="DO"/>
 <pinref part="JP5" gate="G$1" pin="1"/>
-<label x="73.66" y="91.44" size="1.778" layer="95"/>
+<label x="71.12" y="73.66" size="1.778" layer="95"/>
 </segment>
 </net>
@@
 <pinref part="U1" gate="G$1" pin="CD2"/>
 <pinref part="JP7" gate="G$1" pin="1"/>
-<wire x1="63.5" y1="81.28" x2="86.36" y2="81.28" width="0.1524" layer="91"/>
-<label x="73.66" y="81.28" size="1.778" layer="95"/>
+<wire x1="60.96" y1="63.5" x2="83.82" y2="63.5" width="0.1524" layer="91"/>
+<label x="71.12" y="63.5" size="1.778" layer="95"/>
 </segment>
 </net>
@@
 <pinref part="U1" gate="G$1" pin="CD1"/>
 <pinref part="JP6" gate="G$1" pin="1"/>
-<wire x1="63.5" y1="83.82" x2="86.36" y2="83.82" width="0.1524" layer="91"/>
-<label x="73.66" y="83.82" size="1.778" layer="95"/>
+<wire x1="60.96" y1="66.04" x2="83.82" y2="66.04" width="0.1524" layer="91"/>
+<label x="71.12" y="66.04" size="1.778" layer="95"/>
 </segment>
 </net>
@@
 </sheet>
 </sheets>
+<errors>
+</errors>
 </schematic>
 </drawing>
