File: prototyping/microscope/microscope_pcb.brd (EAGLE design)
At the start: 20.1 x 11.7 mm, 7 parts

Commit message: Rename 'board' to 'pcb'
Parts:
- R1: device microscope_board:R0805 -> microscope_pcb:R0805
- SW1, SW2, VOUT+, VOUT-: device microscope_board:1X01 -> microscope_pcb:1X01
- U$1: device microscope_board:DC_DC -> microscope_pcb:DC_DC
- U$2: device microscope_board:USB_CONNECTOR -> microscope_pcb:USB_CONNECTOR
Changed lines of the file:
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@@
 </autorouter>
 <elements>
-<element name="U$1" library="microscope_board" package="DC_DC" value="DC_DC" x="12.68" y="9.76" smashed="yes"/>
-<element name="VOUT+" library="microscope_board" package="1X01" value="" x="5.31" y="9.66" smashed="yes">
+<element name="U$1" library="microscope_pcb" package="DC_DC" value="DC_DC" x="12.68" y="9.76" smashed="yes"/>
+<element name="VOUT+" library="microscope_pcb" package="1X01" value="" x="5.31" y="9.66" smashed="yes">
 <attribute name="VALUE" x="4.04" y="6.485" size="1.27" layer="27"/>
 </element>
-<element name="VOUT-" library="microscope_board" package="1X01" value="" x="1.73" y="9.66" smashed="yes">
+<element name="VOUT-" library="microscope_pcb" package="1X01" value="" x="1.73" y="9.66" smashed="yes">
 <attribute name="VALUE" x="0.46" y="6.485" size="1.27" layer="27"/>
 </element>
-<element name="U$2" library="microscope_board" package="USB_CONNECTOR" value="USB_CONNECTOR" x="10.04" y="4.58" smashed="yes"/>
-<element name="R1" library="microscope_board" package="R0805" value="2K2" x="1.85" y="4.05" smashed="yes" rot="MR270"/>
-<element name="SW1" library="microscope_board" package="1X01" value="" x="18.4" y="2.85" smashed="yes">
+<element name="U$2" library="microscope_pcb" package="USB_CONNECTOR" value="USB_CONNECTOR" x="10.04" y="4.58" smashed="yes"/>
+<element name="R1" library="microscope_pcb" package="R0805" value="2K2" x="1.85" y="4.05" smashed="yes" rot="MR270"/>
+<element name="SW1" library="microscope_pcb" package="1X01" value="" x="18.4" y="2.85" smashed="yes">
 <attribute name="VALUE" x="17.13" y="-0.325" size="1.27" layer="27"/>
 </element>
-<element name="SW2" library="microscope_board" package="1X01" value="" x="18.4" y="5.85" smashed="yes">
+<element name="SW2" library="microscope_pcb" package="1X01" value="" x="18.4" y="5.85" smashed="yes">
 <attribute name="VALUE" x="17.13" y="2.675" size="1.27" layer="27"/>
 </element>
