File: prototyping/microscope/microscope_pcb.sch (EAGLE design)
At the start: 7 parts

Commit message: Rename 'board' to 'pcb'
Parts:
- R1: device microscope_board:R-US_R0805 -> microscope_pcb:R-US_R0805
- SW1, SW2, VOUT+, VOUT-: device microscope_board:PINHD-1X1 -> microscope_pcb:PINHD-1X1
- U$1: device microscope_board:DC_DC -> microscope_pcb:DC_DC
- U$2: device microscope_board:USB_CONNECTOR -> microscope_pcb:USB_CONNECTOR
Changed lines of the file:
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@@
 </classes>
 <parts>
-<part name="U$1" library="microscope_board" deviceset="DC_DC" device=""/>
-<part name="VOUT+" library="microscope_board" deviceset="PINHD-1X1" device=""/>
-<part name="VOUT-" library="microscope_board" deviceset="PINHD-1X1" device=""/>
-<part name="U$2" library="microscope_board" deviceset="USB_CONNECTOR" device=""/>
-<part name="R1" library="microscope_board" deviceset="R-US_" device="R0805" value="2K2"/>
-<part name="SW1" library="microscope_board" deviceset="PINHD-1X1" device=""/>
-<part name="SW2" library="microscope_board" deviceset="PINHD-1X1" device=""/>
+<part name="U$1" library="microscope_pcb" deviceset="DC_DC" device=""/>
+<part name="VOUT+" library="microscope_pcb" deviceset="PINHD-1X1" device=""/>
+<part name="VOUT-" library="microscope_pcb" deviceset="PINHD-1X1" device=""/>
+<part name="U$2" library="microscope_pcb" deviceset="USB_CONNECTOR" device=""/>
+<part name="R1" library="microscope_pcb" deviceset="R-US_" device="R0805" value="2K2"/>
+<part name="SW1" library="microscope_pcb" deviceset="PINHD-1X1" device=""/>
+<part name="SW2" library="microscope_pcb" deviceset="PINHD-1X1" device=""/>
 </parts>
 <sheets>
