File: pmon_log/eagle/pmon_log.brd (EAGLE design)
At the start: 27.9 x 24.1 mm, 29 parts, among them J5 microSD Socket, Q1 16Mhz, U2 LTC2943, U3 TC1015, U4 ATMEGA328TQFP32

Commit message: Added pdf schematic.
Parts:
- removed J5: microSD Socket, SparkFun:MICRO-SD-SOCKET-PP
- added X1: SD-CARD-MSD50, pmon_log:SD_5031821853
Connections:
- new net N$11: X1.MISO
- new net N$12: X1.SCK
- new net N$8: X1.CS
- new net N$9: X1.MOSI
- net +3.3V: now also X1.VCC; no longer J5.4
- net CD: no longer J5.CD1
- net CS: no longer J5.2
- net GND: now also X1.GND; no longer J5.6, J5.GND1, J5.GND3
- net MISO: no longer J5.7
- net MOSI: no longer J5.3
- net SCK: no longer J5.5
Routing:
- net GND: track 23.9 -> 22.4 mm, vias 2 -> 1
Changed lines of the file:
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@@
 <layer number="108" name="tplace-old" color="7" fill="1" visible="yes" active="yes"/>
 <layer number="109" name="ref-old" color="7" fill="1" visible="yes" active="yes"/>
+<layer number="110" name="fp0" color="7" fill="1" visible="yes" active="yes"/>
 <layer number="116" name="Patch_BOT" color="9" fill="4" visible="yes" active="yes"/>
 <layer number="118" name="Rect_Pads" color="7" fill="1" visible="yes" active="yes"/>
+<layer number="120" name="Descript" color="7" fill="1" visible="yes" active="yes"/>
 <layer number="121" name="_tsilk" color="7" fill="1" visible="yes" active="yes"/>
 <layer number="122" name="_bsilk" color="7" fill="1" visible="yes" active="yes"/>
+<layer number="123" name="tTestmark" color="7" fill="1" visible="yes" active="yes"/>
+<layer number="124" name="bTestmark" color="7" fill="1" visible="yes" active="yes"/>
 <layer number="125" name="_tNames" color="7" fill="1" visible="no" active="yes"/>
 <layer number="131" name="prix" color="7" fill="1" visible="yes" active="yes"/>
@@
 <attribute name="VALUE" x="29.972" y="5.588" size="1.27" layer="27" rot="R90"/>
 </element>
-<element name="J5" library="SparkFun" package="MICRO-SD-SOCKET-PP" value="microSD Socket" x="16.129" y="14.478" smashed="yes" rot="R90">
-<attribute name="NAME" x="9.779" y="5.588" size="1.016" layer="25" font="vector" ratio="10" rot="R90"/>
-</element>
 <element name="U$8" library="pmon_log" package="PUSH_BUTTON_GND" value="PUSH_BUTTON_GND" x="2.032" y="19.304" rot="R270"/>
 <element name="J3" library="pmon_log" package="ICSP" value="" x="11.176" y="4.826" rot="MR270"/>
@@
 <element name="R6" library="resistor" package="R0402" value="3K3" x="8.636" y="19.558"/>
 <element name="R7" library="resistor" package="R0402" value="3K3" x="8.636" y="17.78"/>
+<element name="X1" library="pmon_log" package="SD_5031821853" value="SD-CARD-MSD50" x="32.512" y="17.018" rot="R270">
+<attribute name="DIGIKEY" value="WM9750TR-ND" x="32.512" y="17.018" size="1.778" layer="27" rot="R270" display="off"/>
+</element>
 </elements>
 <signals>
@@
 <wire x1="19.304" y1="2.794" x2="18.415" y2="2.794" width="0.3048" layer="1"/>
 <wire x1="18.415" y1="2.794" x2="18.288" y2="2.921" width="0.3048" layer="1"/>
-<contactref element="J5" pad="6"/>
-<contactref element="J5" pad="GND3"/>
-<contactref element="J5" pad="GND1"/>
-<wire x1="6.731" y1="11.049" x2="5.334" y2="11.049" width="0.254" layer="1"/>
-<wire x1="5.334" y1="11.049" x2="5.229" y2="11.038" width="0.254" layer="1"/>
-<via x="6.731" y="11.049" extent="1-16" drill="0.6096"/>
 <contactref element="LED1" pad="C"/>
 <contactref element="LED2" pad="C"/>
+<contactref element="X1" pad="GND"/>
+<wire x1="26.162" y1="21.752" x2="33.312" y2="18.668" width="0" layer="19" extent="1-1"/>
 <wire x1="23.298" y1="19.5326" x2="26.162" y2="21.752" width="0" layer="19" extent="1-1"/>
 <wire x1="21.698" y1="19.5326" x2="23.298" y2="19.5326" width="0" layer="19" extent="1-1"/>
@@
 <wire x1="5.334" y1="22.606" x2="7.874" y2="22.606" width="0" layer="19" extent="1-1"/>
 <wire x1="3.032" y1="21.904" x2="5.334" y2="22.606" width="0" layer="19" extent="1-1"/>
-<wire x1="2.579" y1="14.028" x2="3.032" y2="21.904" width="0" layer="19" extent="1-1"/>
-<wire x1="5.229" y1="11.038" x2="2.579" y2="14.028" width="0" layer="19" extent="1-1"/>
-<wire x1="22.352" y1="11.049" x2="23.298" y2="19.5326" width="0" layer="19" extent="1-1"/>
+<wire x1="4.838" y1="19.558" x2="3.032" y2="21.904" width="0" layer="19" extent="1-1"/>
+<wire x1="4.838" y1="17.78" x2="4.838" y2="19.558" width="0" layer="19" extent="1-1"/>
+<wire x1="22.352" y1="11.049" x2="21.698" y2="19.5326" width="0" layer="19" extent="1-1"/>
 <wire x1="24.095" y1="8.474" x2="22.498" y2="10.9474" width="0" layer="19" extent="1-1"/>
 <wire x1="23.981" y1="1.524" x2="20.863" y2="4.318" width="0" layer="19" extent="1-1"/>
 <wire x1="9.906" y1="2.286" x2="18.288" y2="2.921" width="0" layer="19" extent="1-1"/>
-<wire x1="1.579" y1="0.878" x2="9.906" y2="2.286" width="0" layer="19" extent="1-1"/>
-<wire x1="4.838" y1="19.558" x2="1.579" y2="0.878" width="0" layer="19" extent="1-1"/>
-<wire x1="4.838" y1="17.78" x2="4.838" y2="19.558" width="0" layer="19" extent="1-1"/>
 </signal>
 <signal name="RESET">
@@
 <signal name="SCK">
 <contactref element="U4" pad="17"/>
-<contactref element="J5" pad="5"/>
 <contactref element="J3" pad="SCK"/>
 <wire x1="12.446" y1="4.826" x2="19.298" y2="10.9474" width="0" layer="19" extent="1-1"/>
-<wire x1="5.429" y1="9.938" x2="12.446" y2="4.826" width="0" layer="19" extent="1-1"/>
 </signal>
 <signal name="SER_RX">
@@
 <signal name="MOSI">
 <contactref element="U4" pad="15"/>
-<contactref element="J5" pad="3"/>
 <contactref element="J3" pad="MOSI"/>
 <wire x1="9.906" y1="4.826" x2="17.8054" y2="13.24" width="0" layer="19" extent="1-1"/>
-<wire x1="5.429" y1="7.738" x2="9.906" y2="4.826" width="0" layer="19" extent="1-1"/>
 </signal>
 <signal name="SENSE">
@@
 <signal name="MISO">
 <contactref element="U4" pad="16"/>
-<contactref element="J5" pad="7"/>
 <contactref element="J3" pad="MISO"/>
 <wire x1="12.446" y1="7.366" x2="17.8054" y2="12.44" width="0" layer="19" extent="1-1"/>
-<wire x1="5.429" y1="12.138" x2="12.446" y2="7.366" width="0" layer="19" extent="1-1"/>
 </signal>
 <signal name="+4V">
@@
 </signal>
 <signal name="CS">
-<contactref element="J5" pad="2"/>
 <contactref element="U4" pad="14"/>
-<wire x1="5.829" y1="6.638" x2="17.8054" y2="14.04" width="0" layer="19" extent="1-1"/>
 </signal>
 <signal name="CD">
-<contactref element="J5" pad="CD1"/>
 <contactref element="U4" pad="25"/>
-<wire x1="15.729" y1="12.428" x2="26.3906" y2="12.44" width="0" layer="19" extent="1-1"/>
 </signal>
 <signal name="+VBAT">
@@
 <wire x1="11.43" y1="18.883" x2="17.399" y2="1.143" width="0" layer="19" extent="1-1"/>
 </signal>
-<signal name="+3.3V">
-<contactref element="J5" pad="4"/>
-</signal>
 <signal name="+USB">
 <contactref element="J4" pad="POWER"/>
@@
 <wire x1="9.286" y1="17.78" x2="17.8054" y2="17.24" width="0" layer="19" extent="1-1"/>
 </signal>
+<signal name="N$8">
+<contactref element="X1" pad="CS"/>
+</signal>
+<signal name="N$9">
+<contactref element="X1" pad="MOSI"/>
+</signal>
+<signal name="N$11">
+<contactref element="X1" pad="MISO"/>
+</signal>
+<signal name="N$12">
+<contactref element="X1" pad="SCK"/>
+</signal>
+<signal name="+3.3V">
+<contactref element="X1" pad="VCC"/>
+</signal>
 </signals>
