File: pmon_20v/eagle/pmon_20v.brd (EAGLE design)
At the start: 60 x 60 mm, 34 parts, among them J1 USB, J2 MOLEX 43650-0200, J3 MOLEX 43650-0200, J4 PINHD-2X3, Q1 16Mhz, U1 LTC2943, U2 FT232RL, U3 ATMEGA328TQFP32, U4 TA48M04F

Commit message: Performed final routing.
Parts:
- moved C4 2.00 mm to (53.6, 41.3)
- moved C5 2.00 mm to (53.6, 37.6)
- moved J2 1.00 mm to (42.0, 52.9)
- moved J3 1.00 mm to (53.1, 15.5)
Connections:
- net +5V renamed VIN
Routing:
- net I2C-DATA: track 0.71 -> 38.9 mm, vias 0 -> 2
- net N$1: track 0.32 -> 31.7 mm, vias 0 -> 2
- net I2C-CLK: track 6.87 -> 34.2 mm, vias 0 -> 2
- net VCC: track 107.7 -> 119.6 mm
- net VIN: track 43.4 -> 49.3 mm
- net GND: track 97.2 -> 93.4 mm
- added copper zone on layer 1, net VIN

Commit message: Final tweaks.
Connections:
- net N$22 renamed VOUT
Routing:
- net GND: track 93.4 -> 92.8 mm
- added copper zone on layer 1, net VOUT
Other:
- board text added: "+ VIN -"
- board text added: "+ VOUT -"
- board text added: "VIN 20V 3A MAX"
- board text removed: "+ IN -"
- board text removed: "+ OUT -"
- board text removed: "VIN 20V MAX"
Changed lines of the file:
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@@
 <setting verticaltext="up"/>
 </settings>
-<grid distance="39.3700787" unitdist="mil" unit="mil" style="lines" multiple="1" display="no" altdistance="0.000123031496" altunitdist="mil" altunit="mil"/>
+<grid distance="10" unitdist="mil" unit="mil" style="lines" multiple="1" display="no" altdistance="0.000123031496" altunitdist="mil" altunit="mil"/>
 <layers>
 <layer number="1" name="Top" color="4" fill="1" visible="yes" active="yes"/>
@@
 <wire x1="13.716" y1="9.525" x2="13.716" y2="16.764" width="0.1778" layer="21"/>
 <text x="9.405546875" y="57.41788125" size="1.016" layer="21" font="vector" ratio="10">USB</text>
-<text x="26.931546875" y="54.62388125" size="1.27" layer="21" font="vector" ratio="15">VIN
-20V MAX</text>
+<text x="27.849325" y="52.649709375" size="1.27" layer="21" font="vector" ratio="15">VIN
+20V 3A
+MAX</text>
 <text x="6.87123125" y="28.31666875" size="1.016" layer="21" font="vector" ratio="10" rot="SR270">ICSP</text>
-<text x="15.621" y="2.286" size="1.016" layer="30" font="vector" ratio="15" rot="SMR0" align="bottom-right">POWER-PLAY 20V - REV A
+<text x="15.621" y="2.286" size="1.016" layer="22" font="vector" ratio="15" rot="SMR0" align="bottom-right">POWER-PLAY 20V - REV A
 OSH GITHUB</text>
-<text x="33.281546875" y="50.81388125" size="1.524" layer="21" font="vector" ratio="15">(+)</text>
-<text x="47.886546875" y="50.81388125" size="1.524" layer="21" font="vector" ratio="15">(-)</text>
-<text x="46.616546875" y="11.44388125" size="1.524" layer="21" font="vector" ratio="15">(-)</text>
-<text x="46.616546875" y="17.79388125" size="1.524" layer="21" font="vector" ratio="15">(+)</text>
-<text x="47.251546875" y="7.63388125" size="1.27" layer="21" font="vector" ratio="15">VOUT</text>
-<text x="37.7318" y="50.874503125" size="1.524" layer="22" font="vector" ratio="15" rot="MR180">+ IN -</text>
-<text x="50.531046875" y="20.349059375" size="1.524" layer="22" font="vector" ratio="15" rot="SMR270">+ OUT -</text>
+<text x="37.00886875" y="49.49776875" size="1.524" layer="21" font="vector" ratio="15">(+)</text>
+<text x="44.022190625" y="49.49776875" size="1.524" layer="21" font="vector" ratio="15">(-)</text>
+<text x="50.402078125" y="10.718471875" size="1.524" layer="21" font="vector" ratio="15" rot="R90">(-)</text>
+<text x="50.402078125" y="17.399" size="1.524" layer="21" font="vector" ratio="15" rot="R90">(+)</text>
+<text x="47.62155625" y="13.57468125" size="1.27" layer="21" font="vector" ratio="15" rot="R90">VOUT</text>
+<text x="42.06514375" y="49.831871875" size="1.524" layer="22" font="vector" ratio="15" rot="MR180" align="center">+ VIN -</text>
+<text x="49.65340625" y="15.300540625" size="1.524" layer="22" font="vector" ratio="15" rot="SMR270" align="center">+ VOUT -</text>
 </plain>
 <attributes>
@@
 <param name="mdViaViaSameLayer" value="8mil"/>
 <param name="mnLayersViaInSmd" value="2"/>
-<param name="mdCopperDimension" value="15mil"/>
+<param name="mdCopperDimension" value="25mil"/>
 <param name="mdDrill" value="8mil"/>
 <param name="mdSmdStop" value="0mil"/>
@@
 <via x="10.795" y="45.085" extent="1-16" drill="0.508"/>
 <via x="12.065" y="45.085" extent="1-16" drill="0.508"/>
-<wire x1="4.14" y1="48.346" x2="4.14" y2="46.99" width="0.254" layer="1"/>
-<wire x1="4.14" y1="46.99" x2="4.826" y2="46.99" width="0.254" layer="1"/>
-<wire x1="4.826" y1="46.99" x2="5.08" y2="46.99" width="0.254" layer="1"/>
-<wire x1="5.08" y1="46.99" x2="6.985" y2="46.99" width="0.254" layer="1"/>
-<wire x1="6.985" y1="46.99" x2="7.39" y2="47.395" width="0.254" layer="1"/>
-<wire x1="7.39" y1="47.395" x2="7.39" y2="48.346" width="0.254" layer="1"/>
-<wire x1="5.08" y1="46.99" x2="5.08" y2="45.72" width="0.254" layer="1"/>
-<via x="5.08" y="45.72" extent="1-16" drill="0.508"/>
+<via x="6.096" y="50.466" extent="1-16" drill="0.508"/>
 <wire x1="27.8638" y1="41.0718" x2="27.0256" y2="41.91" width="0.4064" layer="1"/>
 <via x="26.035" y="41.91" extent="1-16" drill="0.508"/>
@@
 <wire x1="29.679" y1="25.654" x2="31.623" y2="25.654" width="0.4064" layer="1"/>
 <wire x1="4.79" y1="48.346" x2="4.826" y2="48.346" width="0.254" layer="1"/>
-<wire x1="4.826" y1="48.346" x2="4.826" y2="46.99" width="0.254" layer="1"/>
 <contactref element="U4" pad="2"/>
 <contactref element="U4" pad="2"/>
@@
 <wire x1="52.832" y1="37.592" x2="52.776" y2="37.592" width="0.254" layer="1"/>
 <wire x1="52.832" y1="37.592" x2="52.776" y2="37.465" width="0.254" layer="1"/>
+<wire x1="4.79" y1="48.346" x2="4.79" y2="49.53" width="0.254" layer="1"/>
+<wire x1="4.14" y1="48.346" x2="4.14" y2="49.53" width="0.254" layer="1"/>
+<wire x1="4.14" y1="49.53" x2="4.79" y2="49.53" width="0.254" layer="1"/>
+<wire x1="7.39" y1="48.346" x2="7.39" y2="49.53" width="0.254" layer="1"/>
+<wire x1="7.39" y1="49.53" x2="6.35" y2="49.53" width="0.254" layer="1"/>
+<wire x1="6.096" y1="49.53" x2="4.79" y2="49.53" width="0.254" layer="1"/>
+<wire x1="6.096" y1="50.466" x2="6.096" y2="49.53" width="0.254" layer="1"/>
+<wire x1="6.096" y1="49.53" x2="6.35" y2="49.53" width="0.254" layer="1"/>
 </signal>
 <signal name="VIN">
@@
 <vertex x="51" y="48"/>
 <vertex x="52" y="47"/>
-<vertex x="52" y="30"/>
-<vertex x="53" y="29"/>
-<vertex x="63" y="29"/>
-<vertex x="63" y="61"/>
+<vertex x="52" y="31"/>
+<vertex x="53" y="30"/>
+<vertex x="53" y="27.519371875"/>
+<vertex x="63" y="27.519371875"/>
+<vertex x="62.780590625" y="52.835384375"/>
+<vertex x="62.945146875" y="61"/>
 </polygon>
 </signal>
@@
 <via x="35.433" y="32.004" extent="1-16" drill="0.3302"/>
 <via x="35.179" y="45.339" extent="1-16" drill="0.3302"/>
-</signal>
-<signal name="N$22">
-<contactref element="R4" pad="I1"/>
-<wire x1="54.958" y1="24.689" x2="54.153" y2="24.689" width="0.4064" layer="1"/>
-<wire x1="54.153" y1="24.689" x2="53.848" y2="24.384" width="0.4064" layer="1"/>
-<contactref element="J3" pad="1"/>
-<wire x1="53.848" y1="24.384" x2="53.975" y2="24.257" width="0.4064" layer="1"/>
-<wire x1="53.975" y1="24.257" x2="53.975" y2="17.899" width="1.524" layer="1"/>
-<wire x1="53.975" y1="17.899" x2="53.07" y2="16.994" width="1.524" layer="1"/>
 </signal>
 <signal name="N$2">
@@
 <signal name="N$4">
 </signal>
+<signal name="VOUT">
+<polygon width="0.4064" layer="1">
+<vertex x="53" y="25"/>
+<vertex x="63" y="25"/>
+<vertex x="63" y="15.5574"/>
+<vertex x="51" y="15.5574"/>
+<vertex x="51" y="22"/>
+<vertex x="53" y="22"/>
+</polygon>
+<contactref element="R4" pad="I1"/>
+<wire x1="54.958" y1="24.689" x2="54.153" y2="24.689" width="0.4064" layer="1"/>
+<wire x1="54.153" y1="24.689" x2="53.848" y2="24.384" width="0.4064" layer="1"/>
+<contactref element="J3" pad="1"/>
+<wire x1="53.848" y1="24.384" x2="53.975" y2="24.257" width="0.4064" layer="1"/>
+<wire x1="53.975" y1="24.257" x2="53.975" y2="17.899" width="1.524" layer="1"/>
+<wire x1="53.975" y1="17.899" x2="53.07" y2="16.994" width="1.524" layer="1"/>
+</signal>
 </signals>

Commit message: Added covers for pmon 20V
Parts:
- C1: value 1uF -> 1uF 50V
Changed lines of the file:
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@@
 <attribute name="NAME" x="52.777015625" y="35.174365625" size="1.016" layer="25" font="vector" ratio="10"/>
 </element>
-<element name="C1" library="pmon_20v" package="C0603" value="1uF" x="47.879" y="28.575" smashed="yes" rot="R180">
+<element name="C1" library="pmon_20v" package="C0603" value="1uF 50V" x="47.879" y="28.575" smashed="yes" rot="R180">
 <attribute name="NAME" x="46.816540625" y="30.004034375" size="1.016" layer="25" font="vector" ratio="10"/>
 </element>
